File: Revision A/zzh.brd (EAGLE design)
At the start: 34.4 x 13.8 mm, 35 parts, among them Y1 32.768KHz, Y2 48.000MHz

Commit message: Revision A, Draft 2 check-in
Parts:
- added L4: (no value), ok-discretes-dev:_PKG_L_0402
- added R1: (no value), ok-discretes-dev:_PKG_C_0402
- moved C14 0.25 mm to (17.5, 2.03)
- moved R2 0.25 mm to (19.6, 2.03)
- moved C7 0.25 mm to (18.5, 2.03)
- moved C16 0.13 mm to (15.2, 8.38)
- moved LED2 0.05 mm to (28.6, 1.02)
- moved R8 0.05 mm to (26.2, 1.02)
Connections:
- new net N$1: L4.1, MOD1.USB_SHIELD_1, MOD1.USB_SHIELD_2
- net BSL: now also R1.2
- net GND: now also L4.2, R1.1; no longer MOD1.USB_SHIELD_1, MOD1.USB_SHIELD_2
Routing:
- net VDDR: track 21.6 -> 11.7 mm, vias 11 -> 5
- net N$1: track 0.00 -> 3.37 mm
- net BSL: track 15.7 -> 18.3 mm
- net VCC: track 21.9 -> 20.2 mm, vias 9 -> 8
- net VDDS: track 16.0 -> 14.7 mm, vias 14 -> 7
- net RESET: track 26.7 -> 25.4 mm
- net GND: track 1.45 -> 0.55 mm, vias 77 -> 83
- net LED: track 12.5 -> 13.1 mm
- added copper zone on layer 2, net GND
- added copper zone on layer 16, net N$2
- removed copper zone on layer 16, net GND
Other:
- board text added: "DRAFT 2 - not tested"
- board text added: "zig-a-zig-ah!"
- board text removed: "DRAFT 1 - not tested"
- board text removed: "zig-ah-zig-ah!"

Commit message: Revision A, Draft 3 check-in
Parts:
- C1, C2: value (none) -> 100n
- C19, C20, R1: value (none) -> DNP
- D2: value RTR5V0U2F -> PRTR5V0U2F,115
- IC1: value (none) -> CC2652R1FRGZ
- IC3: value (none) -> ME6211C33R5G
- SW1: value (none) -> K2-1177SW-D4DW-06
- U1: value (none) -> CH340E
- moved R1 0.33 mm to (10.7, 9.19)
- moved L4 0.05 mm to (5.92, 12.3)
Connections:
- net GND: no longer R1.1
- net VCC: now also R1.1
Routing:
- net VUSB: track 13.4 -> 14.2 mm
- net VCC: track 20.2 -> 20.9 mm
- net PC_TX: track 22.0 -> 21.3 mm
Other:
- board text added: "DRAFT 3 - Untested design!"
- board text added: "zzh!"
- board text removed: "DRAFT 2 - not tested"
