File: Revision A/zzh.sch (EAGLE design)
At the start: 35 parts, among them Y1 32.768KHz, Y2 48.000MHz

Commit message: Revision A, Draft 2 check-in
Parts:
- added L4: (no value), ok-discretes-dev:INDUCTOR-0402
- added R1: (no value), ok-discretes-dev:RES-0402
Connections:
- new net N$1: L4.1, MOD1G$1.USB_SHIELD@1, MOD1G$1.USB_SHIELD@2
- net BSL: now also R1.2
- net GND: now also L4.2, R1.1; no longer MOD1G$1.USB_SHIELD@1, MOD1G$1.USB_SHIELD@2
Other:
- note added: "BSL Trigger button and GP LED TODO: Double check default BSL pin/pd"
- note added: "CC2652R or CC2652RB"
- note added: "DRAFT 2"
- note added: "Draft 2"
- note added: "Revision A DRAFT 2"
- note removed: "BSL Trigger button and GP LED TODO: Double check BSL and LED pins"
- note removed: "CC2652R or CC2652P"
- note removed: "DRAFT 1"
- note removed: "Revision A DRAFT 1"
Changed lines of the file:
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@@
 <layer number="95" name="Names" color="7" fill="1" visible="yes" active="yes"/>
 <layer number="96" name="Values" color="7" fill="1" visible="yes" active="yes"/>
-<layer number="97" name="Info" color="7" fill="1" visible="yes" active="yes"/>
+<layer number="97" name="Info" color="59" fill="1" visible="yes" active="yes"/>
 <layer number="98" name="Guide" color="6" fill="1" visible="yes" active="yes"/>
 <layer number="99" name="SpiceOrder" color="7" fill="1" visible="no" active="yes"/>
@@
 <part name="MOD1" library="ok-modules-dev" deviceset="ZZH_MODULE" device=""/>
 <part name="GND30" library="supply1" library_urn="urn:adsk.eagle:library:371" deviceset="GND" device=""/>
+<part name="R1" library="ok-discretes-dev" deviceset="RES" device="-0402"/>
+<part name="L4" library="ok-discretes-dev" deviceset="INDUCTOR" device="-0402"/>
+<part name="GND31" library="supply1" library_urn="urn:adsk.eagle:library:371" deviceset="GND" device=""/>
 </parts>
 <sheets>
@@
 <text x="165.1" y="15.24" size="2.54" layer="94">zig-a-zig-ah!!
 http://electrolama.com/p/zzh</text>
-<text x="217.17" y="20.32" size="2.54" layer="94">Revision A DRAFT 1</text>
+<text x="217.17" y="20.32" size="2.54" layer="94">Revision A DRAFT 2</text>
 <text x="27.94" y="109.22" size="1.778" layer="91">CC_RXD</text>
 <text x="27.94" y="106.68" size="1.778" layer="91">CC_TXD</text>
@@
 <text x="182.88" y="60.96" size="2.794" layer="91">3V3 LDO</text>
 <text x="12.7" y="50.8" size="2.794" layer="91">USB Serial</text>
-<text x="12.7" y="165.1" size="2.794" layer="91">CC2652R or CC2652P</text>
+<text x="12.7" y="165.1" size="2.794" layer="91">CC2652R or CC2652RB</text>
 <text x="127" y="139.7" size="2.794" layer="91">Balun &amp; Pi Filter for
 SMA Antenna</text>
 <text x="12.7" y="63.5" size="2.794" layer="91">BSL Trigger button and GP LED
-TODO: Double check BSL and LED pins</text>
-<text x="101.6" y="162.56" size="7.62" layer="91">DRAFT 1</text>
+TODO: Double check default BSL pin/pd</text>
+<text x="101.6" y="162.56" size="7.62" layer="91">DRAFT 2</text>
 <text x="7.62" y="12.7" size="2.794" layer="91">Reference Designs:</text>
 <text x="10.16" y="5.08" size="2.286" layer="91">http://www.ti.com/tool/LAUNCHXL-CC26X2R1
 http://www.ti.com/tool/TIDA-010012</text>
+<wire x1="5.08" y1="40.64" x2="15.24" y2="40.64" width="0.1524" layer="97" style="shortdash"/>
+<wire x1="15.24" y1="40.64" x2="15.24" y2="25.4" width="0.1524" layer="97" style="shortdash"/>
+<wire x1="15.24" y1="25.4" x2="5.08" y2="25.4" width="0.1524" layer="97" style="shortdash"/>
+<wire x1="5.08" y1="25.4" x2="5.08" y2="40.64" width="0.1524" layer="97" style="shortdash"/>
+<wire x1="38.1" y1="86.36" x2="38.1" y2="71.12" width="0.1524" layer="97" style="shortdash"/>
+<wire x1="38.1" y1="71.12" x2="48.26" y2="71.12" width="0.1524" layer="97" style="shortdash"/>
+<wire x1="48.26" y1="71.12" x2="48.26" y2="86.36" width="0.1524" layer="97" style="shortdash"/>
+<wire x1="48.26" y1="86.36" x2="38.1" y2="86.36" width="0.1524" layer="97" style="shortdash"/>
+<text x="38.1" y="88.9" size="1.778" layer="97">Draft 2</text>
+<text x="5.08" y="43.18" size="1.778" layer="97">Draft 2</text>
+<wire x1="30.48" y1="170.18" x2="30.48" y2="162.56" width="0.1524" layer="97" style="shortdash"/>
+<wire x1="30.48" y1="162.56" x2="53.34" y2="162.56" width="0.1524" layer="97" style="shortdash"/>
+<wire x1="53.34" y1="162.56" x2="53.34" y2="170.18" width="0.1524" layer="97" style="shortdash"/>
+<wire x1="53.34" y1="170.18" x2="30.48" y2="170.18" width="0.1524" layer="97" style="shortdash"/>
+<text x="30.48" y="172.72" size="1.778" layer="97">Draft 2</text>
 </plain>
 <instances>
@@
 <attribute name="VALUE" x="20.32" y="132.08" size="1.778" layer="96"/>
 </instance>
-<instance part="GND21" gate="1" x="10.16" y="25.4" smashed="yes">
-<attribute name="VALUE" x="7.62" y="22.86" size="1.778" layer="96"/>
+<instance part="GND21" gate="1" x="10.16" y="22.86" smashed="yes">
+<attribute name="VALUE" x="7.62" y="20.32" size="1.778" layer="96"/>
 </instance>
 <instance part="GND22" gate="1" x="58.42" y="25.4" smashed="yes">
@@
 </instance>
 <instance part="SW1" gate="G$1" x="33.02" y="81.28" smashed="yes">
-<attribute name="NAME" x="36.195" y="84.455" size="1.27" layer="95"/>
+<attribute name="NAME" x="28.575" y="76.835" size="1.27" layer="95"/>
 <attribute name="VALUE" x="36.195" y="83.185" size="1.27" layer="96"/>
 </instance>
@@
 <instance part="GND30" gate="1" x="111.76" y="76.2" smashed="yes">
 <attribute name="VALUE" x="106.68" y="73.66" size="1.778" layer="96"/>
+</instance>
+<instance part="R1" gate="G$1" x="43.18" y="78.74" smashed="yes" rot="R90">
+<attribute name="NAME" x="45.72" y="78.74" size="1.778" layer="95"/>
+<attribute name="VALUE" x="46.482" y="74.93" size="1.778" layer="96" rot="R90"/>
+</instance>
+<instance part="L4" gate="G$1" x="10.16" y="30.48" smashed="yes" rot="R270">
+<attribute name="NAME" x="12.7" y="29.21" size="1.778" layer="95"/>
+<attribute name="VALUE" x="7.62" y="33.02" size="1.778" layer="96" rot="R270"/>
+</instance>
+<instance part="GND31" gate="1" x="43.18" y="73.66" smashed="yes">
+<attribute name="VALUE" x="40.64" y="71.12" size="1.778" layer="96"/>
 </instance>
 </instances>
@@
 </segment>
 <segment>
-<pinref part="GND21" gate="1" pin="GND"/>
-<wire x1="10.16" y1="27.94" x2="10.16" y2="35.56" width="0.1524" layer="91"/>
-<wire x1="10.16" y1="35.56" x2="10.16" y2="38.1" width="0.1524" layer="91"/>
-<wire x1="10.16" y1="38.1" x2="12.7" y2="38.1" width="0.1524" layer="91"/>
-<wire x1="12.7" y1="35.56" x2="10.16" y2="35.56" width="0.1524" layer="91"/>
-<junction x="10.16" y="35.56"/>
-<pinref part="MOD1" gate="G$1" pin="USB_SHIELD@1"/>
-<pinref part="MOD1" gate="G$1" pin="USB_SHIELD@2"/>
-</segment>
-<segment>
 <wire x1="55.88" y1="30.48" x2="58.42" y2="30.48" width="0.1524" layer="91"/>
 <pinref part="GND22" gate="1" pin="GND"/>
@@
 <junction x="111.76" y="81.28"/>
 </segment>
+<segment>
+<pinref part="GND21" gate="1" pin="GND"/>
+<wire x1="10.16" y1="25.4" x2="10.16" y2="27.94" width="0.1524" layer="91"/>
+<pinref part="L4" gate="G$1" pin="2"/>
+</segment>
+<segment>
+<pinref part="R1" gate="G$1" pin="1"/>
+<pinref part="GND31" gate="1" pin="GND"/>
+</segment>
 </net>
 <net name="DCOUPL" class="0">
@@
 <segment>
 <pinref part="IC1" gate="G$1" pin="DIO_13"/>
-<wire x1="38.1" y1="81.28" x2="50.8" y2="81.28" width="0.1524" layer="91"/>
-<label x="43.18" y="81.28" size="1.778" layer="95"/>
+<wire x1="38.1" y1="81.28" x2="43.18" y2="81.28" width="0.1524" layer="91"/>
+<label x="45.72" y="81.28" size="1.778" layer="95"/>
 <pinref part="SW1" gate="G$1" pin="2_1"/>
 <pinref part="SW1" gate="G$1" pin="2_2"/>
+<wire x1="43.18" y1="81.28" x2="50.8" y2="81.28" width="0.1524" layer="91"/>
 <wire x1="38.1" y1="78.74" x2="38.1" y2="81.28" width="0.1524" layer="91"/>
 <junction x="38.1" y="81.28"/>
+<pinref part="R1" gate="G$1" pin="2"/>
+<junction x="43.18" y="81.28"/>
 </segment>
 </net>
@@
 </segment>
 </net>
+<net name="N$1" class="0">
+<segment>
+<pinref part="MOD1" gate="G$1" pin="USB_SHIELD@1"/>
+<wire x1="12.7" y1="38.1" x2="10.16" y2="38.1" width="0.1524" layer="91"/>
+<wire x1="10.16" y1="38.1" x2="10.16" y2="35.56" width="0.1524" layer="91"/>
+<pinref part="MOD1" gate="G$1" pin="USB_SHIELD@2"/>
+<wire x1="10.16" y1="35.56" x2="10.16" y2="33.02" width="0.1524" layer="91"/>
+<wire x1="12.7" y1="35.56" x2="10.16" y2="35.56" width="0.1524" layer="91"/>
+<junction x="10.16" y="35.56"/>
+<pinref part="L4" gate="G$1" pin="1"/>
+</segment>
+</net>

Commit message: Revision A, Draft 3 check-in
Parts:
- C1, C2: value (none) -> 100n
- C19, C20, R1: value (none) -> DNP
- D2: value RTR5V0U2F -> PRTR5V0U2F,115
- IC1: value (none) -> CC2652R1FRGZ
- IC3: value (none) -> ME6211C33R5G
- SW1: value (none) -> K2-1177SW-D4DW-06
- U1: value (none) -> CH340E
Connections:
- net GND: no longer R1.1
- net VCC: now also R1.1
Other:
- note added: "BSL Trigger button and general purpose LED"
- note added: "DRAFT 3 Untested design!"
- note added: "Licensed under the Solderpad Hardware License 2.0."
- note added: "Revision A DRAFT 3"
- note added: "Use 1x3 and 1x2 strips of 1.27mm headers for debug"
- note removed: "BSL Trigger button and GP LED TODO: Double check default BSL pin/pd"
- note removed: "DRAFT 2"
- note removed: "Draft 2"
- note removed: "Revision A DRAFT 2"
- moved on the sheet: C10, C7, C8, C9, CON1, IC1, LED2, MOD1G$2, R1, R2, R8, SW1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
