File: zzh/Revision A/zzh.sch (EAGLE design)
At the start: 37 parts, among them IC1 CC2652R1FRGZ, IC3 ME6211C33R5G, SW1 K2-1177SW-D4DW-06, U1 CH340E, Y1 32.768KHz, Y2 48.000MHz

Commit message: zzh: Revision A release
Parts:
- removed C19, C20: DNP, ok-discretes-dev:CAP-0402
- removed CON1: (no value), ok-testdebug-dev:DEBUG_CORTEX-SWD-5PIN-CUT5
- removed L4: (no value), ok-discretes-dev:INDUCTOR-0402
- removed R8: (no value), ok-discretes-dev:RES-0402
- removed U1: CH340E, ok-chips-dev:INTERFACE-CH340E
- added C5: 100n, ok-discretes-dev:CAP-0402
- added C6: 12p, ok-discretes-dev:CAP-0402
- added CON3: DNP, ok-testdebug-dev:DEBUG_CORTEX-SWD/CJTAG-5PIN-CUT5
- added IC2: ME6211C33R5G, ok-chips-dev:POWER-LDO-ME6211C33R5G
- added R3: 100K, ok-discretes-dev:RES-0402
- C10, C9: value 12p -> DNP
- C14: value 100n -> 22u; device ok-discretes-dev:CAP-0402 -> ok-discretes-dev:CAP-0805
- C15: value 22u -> 100n; device ok-discretes-dev:CAP-0805 -> ok-discretes-dev:CAP-0402
- C7: value 100n -> 12p
- IC1: value CC2652R1FRGZ -> CH340E; device ok-chips-dev:WMCU-CC2652R1FRGZ -> ok-chips-dev:INTERFACE-CH340E
- IC3: value ME6211C33R5G -> CC2652R1FRGZ; device ok-chips-dev:POWER-LDO-ME6211C33R5G -> ok-chips-dev:WMCU-CC2652R1FRGZ
- L1: value 6u8 -> BLM18HE152SN1; device ok-discretes-dev:INDUCTOR-0805 -> ok-discretes-dev:INDUCTOR-0603
- L2: value BLM18HE152SN1 -> MLZ2012N6R8LT000; device ok-discretes-dev:INDUCTOR-0603 -> ok-discretes-dev:INDUCTOR-0805
- L3: value (none) -> 0
- R1: value DNP -> 100K
- R2: value 100k -> 100
- Y1: value 32.768KHz -> Q22FA12800150; device ok-xtal-osc-dev:32.768KHZ_Q13FC1350000400 -> ok-xtal-osc-dev:48.000MHZ_CX2016DB48000C0FPLC1
- Y2: value 48.000MHz -> 32.768KHz; device ok-xtal-osc-dev:48.000MHZ_CX2016DB48000C0FPLC1 -> ok-xtal-osc-dev:32.768KHZ_Q13FC1350000400
- renumbered D2 to D1, LED2 to LED1
Connections:
- removed net N$1: L4.1, MOD1G$1.USB_SHIELD@1, MOD1G$1.USB_SHIELD@2
- net ANT: now also C10.2; no longer C20.2
- net BSL: now also IC3.DIO_13, R3.2; no longer IC1.DIO_13, R1.2
- net DCDC_SW: now also IC3.DCDC_SW, L2.1; no longer IC1.DCDC_SW, L1.1
- net DCOUPL: now also IC3.DCOUPL; no longer IC1.DCOUPL
- net GND: now also C5.1, C6.1, CON3.GND@3, IC1.GND, IC2.GND, IC3.EP, MOD1G$1.USB_SHIELD@1, MOD1G$1.USB_SHIELD@2, Y1.2, Y1.4; no longer C19.1, C20.1, CON1.GND@3, IC1.EP, IC3.GND, L4.2, U1.GND, Y2.2, Y2.4
- net LED: now also IC3.DIO_7, R2.1; no longer IC1.DIO_7, R8.1
- net N$16: now also R2.2; no longer R8.2
- net PC_RX: now also IC1.RXD, IC3.DIO_3; no longer IC1.DIO_3, U1.RXD
- net PC_TX: now also IC1.TXD, IC3.DIO_2; no longer IC1.DIO_2, U1.TXD
- net RESET: now also C5.2, CON3.NRESET, IC3.RESET_N, R1.1; no longer C7.2, CON1.NRESET, IC1.RESET_N, R2.1
- net RF_N: now also IC3.RF_N; no longer IC1.RF_N
- net RF_P: now also IC3.RF_P; no longer IC1.RF_P
- net TCK: now also CON3.SWDCLK/TCK, IC3.JTAG_TCKC; no longer CON1.SWDCLK(TCK), IC1.JTAG_TCKC
- net TMS: now also CON3.SWDIO/TMS, IC3.JTAG_TMSC; no longer CON1.SWDIO/(TMS), IC1.JTAG_TMSC
- net UD+: now also IC1.UD+; no longer U1.UD+
- net UD-: now also IC1.UD-; no longer U1.UD-
- net UNBAL: now also C9.2; no longer C19.2
- net VCC: now also C4.1, CON3.VCC, IC1.V3, IC1.VCC, IC2.VOUT, L1.1, R1.2, R3.1; no longer C3.1, CON1.VCC, IC3.VOUT, L2.1, R1.1, R2.2, U1.V3, U1.VCC
- net VDDR: now also IC3.VDDR, IC3.VDDR_RF, L2.2; no longer IC1.VDDR, IC1.VDDR_RF, L1.2
- net VDDS: now also IC3.VDDS, IC3.VDDS2, IC3.VDDS3, IC3.VDDS_DCDC, L1.2; no longer IC1.VDDS, IC1.VDDS2, IC1.VDDS3, IC1.VDDS_DCDC, L2.2
- net VUSB: now also C3.1, IC2.EN, IC2.VIN; no longer C4.1, IC3.EN, IC3.VIN
- net X32K_Q1: now also C6.2, IC3.X32K_Q1, Y2.1; no longer C9.2, IC1.X32K_Q1, Y1.1
- net X32K_Q2: now also C7.2, IC3.X32K_Q2, Y2.2; no longer C10.2, IC1.X32K_Q2, Y1.2
- net X48M_N: now also IC3.X48M_N, Y1.3; no longer IC1.X48M_N, Y2.3
- net X48M_P: now also IC3.X48M_P, Y1.1; no longer IC1.X48M_P, Y2.1
Other:
- note added: "(zzh boards ship with CC2652R)"
- note added: "1.27mm 2x3 header Use zzh-debug adapter PCB to convert to standard 2x5 pinout."
- note added: "Balun & Pi Filter"
- note added: "CC2652R / CC2652RB"
- note added: "CON1"
- note added: "CON2"
- note added: "Edge Mount Female SMA"
- note added: "L2 and C16 near pin 33"
- note added: "Revision A"
- note added: "cJTAG Debug"
- note removed: "Balun & Pi Filter for SMA Antenna"
- note removed: "CC2652R or CC2652RB"
- note removed: "DRAFT 3 Untested design!"
- note removed: "L1 and C16 near pin 33"
- note removed: "Revision A DRAFT 3"
- note removed: "SWD Debug"
- note removed: "Use 1x3 and 1x2 strips of 1.27mm headers for debug"
- moved on the sheet: C10, C11, C12, C13, C14, C15, C16, C17, C18, C3, C4, C7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
